File: av3/reles.kicad_sch (KiCad schematic)
At the start: 20 parts, among them J1 Conn_01x03, J2 Conn_01x03, J3 Conn_01x03, J4 Conn_01x03, K1 SANYOU_SRD_Form_C, K2 SANYOU_SRD_Form_C, K3 SANYOU_SRD_Form_C, K4 SANYOU_SRD_Form_C, Q1 BC337, Q2 BC337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

Commit message: FEAT: Adição das footprints dos capacitores (C) e screw_terminals (J)
Parts:
- J1, J2, J3, J4: footprint (none) -> TerminalBlock_Phoenix:TerminalBlock_Phoenix_MKDS-1,5-3_1x03_P5.00mm_Horizontal
Changed lines of the file:
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@@
 			)
 		)
-		(property "Footprint" ""
+		(property "Footprint" "TerminalBlock_Phoenix:TerminalBlock_Phoenix_MKDS-1,5-3_1x03_P5.00mm_Horizontal"
 			(at 173.99 93.98 0)
 			(effects
@@
 			)
 		)
-		(property "Footprint" ""
+		(property "Footprint" "TerminalBlock_Phoenix:TerminalBlock_Phoenix_MKDS-1,5-3_1x03_P5.00mm_Horizontal"
 			(at 173.99 49.53 0)
 			(effects
@@
 			)
 		)
-		(property "Footprint" ""
+		(property "Footprint" "TerminalBlock_Phoenix:TerminalBlock_Phoenix_MKDS-1,5-3_1x03_P5.00mm_Horizontal"
 			(at 97.79 93.98 0)
 			(effects
@@
 			)
 		)
-		(property "Footprint" ""
+		(property "Footprint" "TerminalBlock_Phoenix:TerminalBlock_Phoenix_MKDS-1,5-3_1x03_P5.00mm_Horizontal"
 			(at 97.79 48.26 0)
 			(effects

Commit message: Alteração do footprint do PS1 e inicio da PCB
Parts:
- R2, R3, R4, R5: value 6,2k -> 15k; footprint (none) -> Resistor_THT:R_Axial_DIN0207_L6.3mm_D2.5mm_P7.62mm_Horizontal
Changed lines of the file:
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@@
 			)
 		)
-		(property "Value" "6,2k"
+		(property "Value" "15k"
 			(at 129.54 65.278 90)
 			(effects
@@
 			)
 		)
-		(property "Footprint" ""
+		(property "Footprint" "Resistor_THT:R_Axial_DIN0207_L6.3mm_D2.5mm_P7.62mm_Horizontal"
 			(at 129.54 61.468 90)
 			(effects
@@
 			)
 		)
-		(property "Value" "6,2k"
+		(property "Value" "15k"
 			(at 129.54 109.728 90)
 			(effects
@@
 			)
 		)
-		(property "Footprint" ""
+		(property "Footprint" "Resistor_THT:R_Axial_DIN0207_L6.3mm_D2.5mm_P7.62mm_Horizontal"
 			(at 129.54 105.918 90)
 			(effects
@@
 			)
 		)
-		(property "Value" "6,2k"
+		(property "Value" "15k"
 			(at 53.34 64.008 90)
 			(effects
@@
 			)
 		)
-		(property "Footprint" ""
+		(property "Footprint" "Resistor_THT:R_Axial_DIN0207_L6.3mm_D2.5mm_P7.62mm_Horizontal"
 			(at 53.34 60.198 90)
 			(effects
@@
 			)
 		)
-		(property "Value" "6,2k"
+		(property "Value" "15k"
 			(at 53.34 109.728 90)
 			(effects
@@
 			)
 		)
-		(property "Footprint" ""
+		(property "Footprint" "Resistor_THT:R_Axial_DIN0207_L6.3mm_D2.5mm_P7.62mm_Horizontal"
 			(at 53.34 105.918 90)
 			(effects

Commit message: Mudança de footprints e mudança na PCB
Connections:
- net at J4.1 (Pin_1): now also K4.3; no longer K4.4
- net at J4.3 (Pin_3): now also K4.4; no longer K4.3
- net at K1.3: now also J1.1 (Pin_1); no longer J1.3 (Pin_3)
- net at K1.4: now also J1.3 (Pin_3); no longer J1.1 (Pin_1)
- net at J2.1 (Pin_1): now also K2.3; no longer K2.4
- net at J2.3 (Pin_3): now also K2.4; no longer K2.3
- net at K3.3: now also J3.1 (Pin_1); no longer J3.3 (Pin_3)
- net at K3.4: now also J3.3 (Pin_3); no longer J3.1 (Pin_1)
Changed lines of the file:
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@@
 		(lib_id "Connector_Generic:Conn_01x03")
 		(at 173.99 93.98 0)
-		(unit 1)
-		(exclude_from_sim no)
-		(in_bom yes)
-		(on_board yes)
-		(dnp no)
-		(fields_autoplaced yes)
+		(mirror x)
+		(unit 1)
+		(exclude_from_sim no)
+		(in_bom yes)
+		(on_board yes)
+		(dnp no)
 		(property "Reference" "J4"
-			(at 176.53 92.7099 0)
+			(at 176.53 95.2501 0)
 			(effects
 				(font
@@
 		)
 		(property "Value" "Conn_01x03"
-			(at 176.53 95.2499 0)
+			(at 176.53 92.7101 0)
 			(effects
 				(font
@@
 		(lib_id "Connector_Generic:Conn_01x03")
 		(at 173.99 49.53 0)
-		(unit 1)
-		(exclude_from_sim no)
-		(in_bom yes)
-		(on_board yes)
-		(dnp no)
-		(fields_autoplaced yes)
+		(mirror x)
+		(unit 1)
+		(exclude_from_sim no)
+		(in_bom yes)
+		(on_board yes)
+		(dnp no)
 		(property "Reference" "J2"
-			(at 176.53 48.2599 0)
+			(at 176.53 50.8001 0)
 			(effects
 				(font
@@
 		)
 		(property "Value" "Conn_01x03"
-			(at 176.53 50.7999 0)
+			(at 176.53 48.2601 0)
 			(effects
 				(font
@@
 		(lib_id "Connector_Generic:Conn_01x03")
 		(at 97.79 93.98 0)
-		(unit 1)
-		(exclude_from_sim no)
-		(in_bom yes)
-		(on_board yes)
-		(dnp no)
-		(fields_autoplaced yes)
+		(mirror x)
+		(unit 1)
+		(exclude_from_sim no)
+		(in_bom yes)
+		(on_board yes)
+		(dnp no)
 		(property "Reference" "J3"
-			(at 100.33 92.7099 0)
+			(at 100.33 95.2501 0)
 			(effects
 				(font
@@
 		)
 		(property "Value" "Conn_01x03"
-			(at 100.33 95.2499 0)
+			(at 100.33 92.7101 0)
 			(effects
 				(font
@@
 		(lib_id "Connector_Generic:Conn_01x03")
 		(at 97.79 48.26 0)
-		(unit 1)
-		(exclude_from_sim no)
-		(in_bom yes)
-		(on_board yes)
-		(dnp no)
-		(fields_autoplaced yes)
+		(mirror x)
+		(unit 1)
+		(exclude_from_sim no)
+		(in_bom yes)
+		(on_board yes)
+		(dnp no)
 		(property "Reference" "J1"
-			(at 100.33 46.9899 0)
+			(at 100.33 49.5301 0)
 			(effects
 				(font
@@
 		)
 		(property "Value" "Conn_01x03"
-			(at 100.33 49.5299 0)
-			(effects
-				(font
+			(at 100.33 46.9901 0)
+			(effects
+				(font
