File: av3/modulo_entrada.kicad_sch (KiCad schematic)
At the start: 28 parts, among them J5 Conn_01x02, J6 Conn_01x02, J7 Conn_01x02, J8 Conn_01x02, U2 4N25, U3 4N25, U4 4N25, U5 4N25

Commit message: FEAT: Adição das footprints dos capacitores (C) e screw_terminals (J)
Parts:
- D11, D5, D7, D9: footprint (none) -> LED_SMD:LED_0201_0603Metric
- J5, J6, J7, J8: footprint (none) -> TerminalBlock_Phoenix:TerminalBlock_Phoenix_MKDS-1,5-2_1x02_P5.00mm_Horizontal
Changed lines of the file:
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@@
 			)
 		)
-		(property "Footprint" ""
+		(property "Footprint" "TerminalBlock_Phoenix:TerminalBlock_Phoenix_MKDS-1,5-2_1x02_P5.00mm_Horizontal"
 			(at 111.76 63.5 0)
 			(effects
@@
 			)
 		)
-		(property "Footprint" ""
+		(property "Footprint" "LED_SMD:LED_0201_0603Metric"
 			(at 41.91 102.87 0)
 			(effects
@@
 			)
 		)
-		(property "Footprint" ""
+		(property "Footprint" "TerminalBlock_Phoenix:TerminalBlock_Phoenix_MKDS-1,5-2_1x02_P5.00mm_Horizontal"
 			(at 33.02 63.5 0)
 			(effects
@@
 			)
 		)
-		(property "Footprint" ""
+		(property "Footprint" "LED_SMD:LED_0201_0603Metric"
 			(at 120.65 64.77 0)
 			(effects
@@
 			)
 		)
-		(property "Footprint" ""
+		(property "Footprint" "TerminalBlock_Phoenix:TerminalBlock_Phoenix_MKDS-1,5-2_1x02_P5.00mm_Horizontal"
 			(at 111.76 101.6 0)
 			(effects
@@
 			)
 		)
-		(property "Footprint" ""
+		(property "Footprint" "TerminalBlock_Phoenix:TerminalBlock_Phoenix_MKDS-1,5-2_1x02_P5.00mm_Horizontal"
 			(at 33.02 101.6 0)
 			(effects
@@
 			)
 		)
-		(property "Footprint" ""
+		(property "Footprint" "LED_SMD:LED_0201_0603Metric"
 			(at 120.65 102.87 0)
 			(effects
@@
 			)
 		)
-		(property "Footprint" ""
+		(property "Footprint" "LED_SMD:LED_0201_0603Metric"
 			(at 41.91 64.77 0)
 			(effects

Commit message: Alteração do footprint do PS1 e inicio da PCB
Parts:
- R10, R12, R13, R15, R16, R6, R7, R9: value R -> 100; footprint (none) -> Resistor_THT:R_Axial_DIN0204_L3.6mm_D1.6mm_P5.08mm_Horizontal
Changed lines of the file:
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@@
 			)
 		)
-		(property "Value" "R"
+		(property "Value" "100"
 			(at 49.53 49.53 90)
 			(effects
@@
 			)
 		)
-		(property "Footprint" ""
+		(property "Footprint" "Resistor_THT:R_Axial_DIN0204_L3.6mm_D1.6mm_P5.08mm_Horizontal"
 			(at 49.53 55.118 90)
 			(effects
@@
 			)
 		)
-		(property "Value" "R"
+		(property "Value" "100"
 			(at 128.27 49.53 90)
 			(effects
@@
 			)
 		)
-		(property "Footprint" ""
+		(property "Footprint" "Resistor_THT:R_Axial_DIN0204_L3.6mm_D1.6mm_P5.08mm_Horizontal"
 			(at 128.27 55.118 90)
 			(effects
@@
 			)
 		)
-		(property "Value" "R"
+		(property "Value" "100"
 			(at 44.45 96.5199 0)
 			(effects
@@
 			)
 		)
-		(property "Footprint" ""
+		(property "Footprint" "Resistor_THT:R_Axial_DIN0204_L3.6mm_D1.6mm_P5.08mm_Horizontal"
 			(at 40.132 95.25 90)
 			(effects
@@
 			)
 		)
-		(property "Value" "R"
+		(property "Value" "100"
 			(at 44.45 58.4199 0)
 			(effects
@@
 			)
 		)
-		(property "Footprint" ""
+		(property "Footprint" "Resistor_THT:R_Axial_DIN0204_L3.6mm_D1.6mm_P5.08mm_Horizontal"
 			(at 40.132 57.15 90)
 			(effects
@@
 			)
 		)
-		(property "Value" "R"
+		(property "Value" "100"
 			(at 49.53 87.63 90)
 			(effects
@@
 			)
 		)
-		(property "Footprint" ""
+		(property "Footprint" "Resistor_THT:R_Axial_DIN0204_L3.6mm_D1.6mm_P5.08mm_Horizontal"
 			(at 49.53 93.218 90)
 			(effects
@@
 			)
 		)
-		(property "Value" "R"
+		(property "Value" "100"
 			(at 123.19 96.5199 0)
 			(effects
@@
 			)
 		)
-		(property "Footprint" ""
+		(property "Footprint" "Resistor_THT:R_Axial_DIN0204_L3.6mm_D1.6mm_P5.08mm_Horizontal"
 			(at 118.872 95.25 90)
 			(effects
@@
 			)
 		)
-		(property "Value" "R"
+		(property "Value" "100"
 			(at 128.27 87.63 90)
 			(effects
@@
 			)
 		)
-		(property "Footprint" ""
+		(property "Footprint" "Resistor_THT:R_Axial_DIN0204_L3.6mm_D1.6mm_P5.08mm_Horizontal"
 			(at 128.27 93.218 90)
 			(effects
@@
 			)
 		)
-		(property "Value" "R"
+		(property "Value" "100"
 			(at 123.19 58.4199 0)
 			(effects
@@
 			)
 		)
-		(property "Footprint" ""
+		(property "Footprint" "Resistor_THT:R_Axial_DIN0204_L3.6mm_D1.6mm_P5.08mm_Horizontal"
 			(at 118.872 57.15 90)
 			(effects

Commit message: Mudança de footprints e mudança na PCB
Parts:
- D11, D5, D7, D9: footprint LED_SMD:LED_0201_0603Metric -> LED_THT:LED_D3.0mm
- R10, R12, R13, R15, R16, R6, R7, R9: footprint Resistor_THT:R_Axial_DIN0204_L3.6mm_D1.6mm_P5.08mm_Horizontal -> Resistor_SMD:R_1206_3216Metric_Pad1.30x1.75mm_HandSolder
- R11, R14, R17, R8: footprint (none) -> Resistor_SMD:R_1206_3216Metric_Pad1.30x1.75mm_HandSolder
Connections:
- net at D7.1 (K), U3.2: now also J6.2 (Pin_2); no longer J6.1 (Pin_1)
- net at R10.1, R9.1: now also J6.1 (Pin_1); no longer J6.2 (Pin_2)
- net at D9.1 (K), U4.2: now also J7.2 (Pin_2); no longer J7.1 (Pin_1)
- net at D5.1 (K), U2.2: now also J5.2 (Pin_2); no longer J5.1 (Pin_1)
- net at R6.1, R7.1: now also J5.1 (Pin_1); no longer J5.2 (Pin_2)
- net at D11.1 (K), U5.2: now also J8.2 (Pin_2); no longer J8.1 (Pin_1)
- net at R15.1, R16.1: now also J8.1 (Pin_1); no longer J8.2 (Pin_2)
- net at R12.1, R13.1: now also J7.1 (Pin_1); no longer J7.2 (Pin_2)
Other:
- moved on the sheet: J5, J6, J7, J8

Commit message: Algumas trilhas feitas
Changed lines of the file:
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@@
 	(text "CALCULAR RESISTÊNCIAS"
 		(exclude_from_sim no)
-		(at 98.806 74.422 0)
+		(at 99.822 123.952 0)
 		(effects
 			(font
