File: av3/teclado_matricial.kicad_sch (KiCad schematic)
At the start: 16 parts, among them SW10 SW_MEC_5G, SW11 SW_MEC_5G, SW12 SW_MEC_5G, SW13 SW_MEC_5G, SW14 SW_MEC_5G, SW15 SW_MEC_5G, SW16 SW_MEC_5G, SW17 SW_MEC_5G, SW2 SW_MEC_5G, SW3 SW_MEC_5G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

Commit message: Alteração do footprint do PS1 e inicio da PCB
Parts:
- removed SW10, SW11, SW12, SW13, SW14, SW15, SW16, SW17, SW2, SW3, SW4, SW5, SW6, SW7, SW8, SW9: SW_MEC_5G, symbol Switch:SW_MEC_5G
- added SW10, SW11, SW12, SW13, SW14, SW15, SW16, SW17, SW2, SW3, SW4, SW5, SW6, SW7, SW8, SW9: SW_Omron_B3FS, Button_Switch_SMD:SW_Push_1P1T_NO_CK_KSC7xxJ, symbol Switch:SW_Omron_B3FS
Connections:
- net C1: now also SW10.2, SW14.2, SW2.2, SW6.2
- net C2: now also SW11.2, SW15.2, SW3.2, SW7.2
- net C3: now also SW12.2, SW16.2, SW4.2, SW8.2
- net C4: now also SW13.2, SW17.2, SW5.2, SW9.2
- net L1: now also SW2.1, SW3.1, SW4.1, SW5.1
- net L2: now also SW6.1, SW7.1, SW8.1, SW9.1
- net L3: now also SW10.1, SW11.1, SW12.1, SW13.1
- net L4: now also SW14.1, SW15.1, SW16.1, SW17.1

Commit message: Algumas trilhas feitas
Connections:
- net C1: now also SW13.2, SW17.2, SW5.2, SW9.2; no longer SW10.2, SW14.2, SW2.2, SW6.2
- net C2: now also SW12.2, SW16.2, SW4.2, SW8.2; no longer SW11.2, SW15.2, SW3.2, SW7.2
- net C3: now also SW11.2, SW15.2, SW3.2, SW7.2; no longer SW12.2, SW16.2, SW4.2, SW8.2
- net C4: now also SW10.2, SW14.2, SW2.2, SW6.2; no longer SW13.2, SW17.2, SW5.2, SW9.2
Changed lines of the file:
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@@
 		)
 	)
-	(global_label "C3"
+	(global_label "C2"
 		(shape input)
 		(at 97.79 58.42 90)
@@
 		)
 	)
-	(global_label "C4"
+	(global_label "C1"
 		(shape input)
 		(at 113.03 58.42 90)
@@
 		)
 	)
-	(global_label "C1"
+	(global_label "C4"
 		(shape input)
 		(at 67.31 58.42 90)
@@
 		)
 	)
-	(global_label "C2"
+	(global_label "C3"
 		(shape input)
 		(at 82.55 58.42 90)
