File: av3/av3.kicad_pcb (KiCad board)
At the start: 2 copper layers, 108 parts, among them J1 Conn_01x03, J10 Conn_01x03, J11 DE9_Pins_MountingHoles, J12 Conn_01x03, J13 Conn_01x03, J14 Conn_01x03, J15 Conn_02x04_Odd_Even, J16 Screw_Terminal_01x03, J2 Conn_01x03, J3 Conn_01x03, J4 Conn_01x03, J5 Conn_01x02, J6 Conn_01x02, J7 Conn_01x02, J8 Conn_01x02, J9 Conn_02x05_Odd_Even, K1 SANYOU_SRD_Form_C, K2 SANYOU_SRD_Form_C, K3 SANYOU_SRD_Form_C, K4 SANYOU_SRD_Form_C, Q1 BC337, Q2 BC337, Q3 BC337, Q4 BC337, SW1 SW_MEC_5G, SW10 SW_Omron_B3FS, SW11 SW_Omron_B3FS, SW12 SW_Omron_B3FS, SW13 SW_Omron_B3FS, SW14 SW_Omron_B3FS, SW15 SW_Omron_B3FS, SW16 SW_Omron_B3FS, SW17 SW_Omron_B3FS, SW2 SW_Omron_B3FS, SW3 SW_Omron_B3FS, SW4 SW_Omron_B3FS, SW5 SW_Omron_B3FS, SW6 SW_Omron_B3FS, SW7 SW_Omron_B3FS, SW8 SW_Omron_B3FS, SW9 SW_Omron_B3FS, U1 ATmega2560-16A, U10 LCD-016N002L, U2 4N25, U3 4N25, U4 4N25, U5 4N25, U6 TL084, U7 6N137, U8 6N137, U9 MAX232, Y1 16Mhz

Commit message: Mudança de footprints e mudança na PCB
Parts:
- added R11: R, Resistor_SMD:R_1206_3216Metric_Pad1.30x1.75mm_HandSolder, F.Cu at (-161.4, 231.2)
- added R14: R, Resistor_SMD:R_1206_3216Metric_Pad1.30x1.75mm_HandSolder, F.Cu at (-146.5, 231.2)
- added R17: R, Resistor_SMD:R_1206_3216Metric_Pad1.30x1.75mm_HandSolder, F.Cu at (-130.8, 231.4)
- added R18: 10K, Resistor_THT:R_Axial_DIN0207_L6.3mm_D2.5mm_P7.62mm_Horizontal, F.Cu at (15.2, 354.9)
- added R19: 10K, Resistor_THT:R_Axial_DIN0207_L6.3mm_D2.5mm_P7.62mm_Horizontal, F.Cu at (23.0, 350.3)
- added R20: 10K, Resistor_THT:R_Axial_DIN0207_L6.3mm_D2.5mm_P7.62mm_Horizontal, F.Cu at (20.2, 337.3)
- added R21: 10K, Resistor_THT:R_Axial_DIN0207_L6.3mm_D2.5mm_P7.62mm_Horizontal, F.Cu at (20.2, 332.6)
- added R8: R, Resistor_SMD:R_1206_3216Metric_Pad1.30x1.75mm_HandSolder, F.Cu at (-176.2, 231.2)
- D11, D5, D7, D9: footprint LED_SMD:LED_0201_0603Metric -> LED_THT:LED_D3.0mm
- J10, J12, J13, J14: footprint TerminalBlock_Phoenix:TerminalBlock_Phoenix_MKDS-1,5-3_1x03_P5.00mm_Horizontal -> Connector_PinHeader_2.54mm:PinHeader_1x03_P2.54mm_Vertical
- J15: footprint Connector_PinHeader_2.54mm:PinHeader_2x04_P2.54mm_Vertical -> Connector_IDC:IDC-Header_2x04_P2.54mm_Vertical
- R10, R12, R13, R15, R16, R6, R7, R9: footprint Resistor_THT:R_Axial_DIN0204_L3.6mm_D1.6mm_P5.08mm_Horizontal -> Resistor_SMD:R_1206_3216Metric_Pad1.30x1.75mm_HandSolder; moved to B.Cu
- RV1, RV2, RV3, RV4, RV5: footprint Resistor_THT:R_Axial_DIN0207_L6.3mm_D2.5mm_P7.62mm_Horizontal -> Potentiometer_THT:Potentiometer_Bourns_3296W_Vertical
- U6: footprint Connector_PinHeader_2.54mm:PinHeader_2x04_P2.54mm_Vertical -> Package_DIP:DIP-14_W7.62mm
- moved J10 355.9 mm to (-18.9, 360.8)
- moved RV1 348.6 mm to (-29.9, 350.6), turned to 90 degrees
- moved RV2 344.7 mm to (-22.8, 350.6), turned to 90 degrees
- moved J12 344.2 mm to (-15.2, 360.8)
- moved RV3 341.0 mm to (-15.6, 350.6), turned to 90 degrees
- moved RV4 337.4 mm to (-8.60, 350.6), turned to 90 degrees
- moved J15 336.1 mm to (36.7, 347.0), turned to 180 degrees
- moved J13 332.5 mm to (-11.5, 360.8)
- moved U6 330.4 mm to (2.37, 347.6), turned to 90 degrees
- moved J14 320.9 mm to (-7.80, 360.8)
- moved J5 270.6 mm to (-180.5, 264.7)
- moved J6 269.8 mm to (-165.6, 264.7)
- moved J7 269.0 mm to (-150.7, 264.7)
- moved J8 268.2 mm to (-135.4, 264.8)
- moved R6 256.6 mm to (-180.5, 250.7), turned to 90 degrees
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Connections:
- J5 pad 1: Net-(D5-K) -> Net-(J5-Pin_1)
- J5 pad 2: Net-(J5-Pin_2) -> Net-(D5-K)
- J6 pad 1: Net-(D7-K) -> Net-(J6-Pin_1)
- J6 pad 2: Net-(J6-Pin_2) -> Net-(D7-K)
- J7 pad 1: Net-(D9-K) -> Net-(J7-Pin_1)
- J7 pad 2: Net-(J7-Pin_2) -> Net-(D9-K)
- J8 pad 1: Net-(D11-K) -> Net-(J8-Pin_1)
- J8 pad 2: Net-(J8-Pin_2) -> Net-(D11-K)
- K1 pad 3: Net-(J1-Pin_3) -> Net-(J1-Pin_1)
- K1 pad 4: Net-(J1-Pin_1) -> Net-(J1-Pin_3)
- K2 pad 3: Net-(J2-Pin_3) -> Net-(J2-Pin_1)
- K2 pad 4: Net-(J2-Pin_1) -> Net-(J2-Pin_3)
- K3 pad 3: Net-(J3-Pin_3) -> Net-(J3-Pin_1)
- K3 pad 4: Net-(J3-Pin_1) -> Net-(J3-Pin_3)
- K4 pad 3: Net-(J4-Pin_3) -> Net-(J4-Pin_1)
- K4 pad 4: Net-(J4-Pin_1) -> Net-(J4-Pin_3)
- R10 pad 1: Net-(J6-Pin_2) -> Net-(J6-Pin_1)
- R12 pad 1: Net-(J7-Pin_2) -> Net-(J7-Pin_1)
- R13 pad 1: Net-(J7-Pin_2) -> Net-(J7-Pin_1)
- R15 pad 1: Net-(J8-Pin_2) -> Net-(J8-Pin_1)
- R16 pad 1: Net-(J8-Pin_2) -> Net-(J8-Pin_1)
- R6 pad 1: Net-(J5-Pin_2) -> Net-(J5-Pin_1)
- R7 pad 1: Net-(J5-Pin_2) -> Net-(J5-Pin_1)
- R9 pad 1: Net-(J6-Pin_2) -> Net-(J6-Pin_1)
Routing:
- net in0.4: track 0.00 -> 61.9 mm
- net in0.1: track 0.00 -> 61.2 mm
- net in0.3: track 0.00 -> 55.2 mm
- net in0.2: track 0.00 -> 55.2 mm
- net q0.1: track 0.00 -> 54.7 mm
- net q0.4: track 0.00 -> 48.7 mm
- net q0.2: track 0.00 -> 39.6 mm
- net q0.3: track 0.00 -> 36.9 mm
- net Net-(J2-Pin_2): track 0.00 -> 25.8 mm
- net Net-(J4-Pin_2): track 0.00 -> 25.8 mm
- net Net-(J3-Pin_2): track 0.00 -> 25.8 mm
- net Net-(J1-Pin_2): track 0.00 -> 25.7 mm
- net +5V: track 21.6 -> 46.7 mm
- net Net-(D5-K): track 0.00 -> 19.8 mm
- net Net-(D9-K): track 0.00 -> 19.8 mm
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Other:
- board outline added: 180 x 180 mm
- board text added: "K"
- board text removed: "CRISTAL"

Commit message: Algumas trilhas feitas
Parts:
- added C6: 100nF, Capacitor_THT:CP_Radial_D4.0mm_P1.50mm, F.Cu at (-147.7, 161.8)
- added C7: 100nF, Capacitor_THT:CP_Radial_D4.0mm_P1.50mm, F.Cu at (-142.6, 161.0)
- added C8: 100nF, Capacitor_THT:CP_Radial_D4.0mm_P1.50mm, F.Cu at (-142.6, 147.3)
- added C9: 100nF, Capacitor_THT:CP_Radial_D4.0mm_P1.50mm, F.Cu at (-147.7, 147.4)
- moved U10 318.1 mm to (-114.6, 94.2)
- moved SW10 269.4 mm to (-239.9, 144.5)
- moved SW11 269.4 mm to (-231.5, 144.5)
- moved SW12 269.4 mm to (-223.1, 144.5)
- moved SW14 269.4 mm to (-239.9, 153.8)
- moved SW15 269.4 mm to (-231.5, 153.8)
- moved SW16 269.4 mm to (-223.1, 153.8)
- moved SW2 269.4 mm to (-239.9, 125.9)
- moved SW3 269.4 mm to (-231.5, 125.9)
- moved SW4 269.4 mm to (-223.1, 125.9)
- moved SW6 269.4 mm to (-239.9, 135.2)
- moved SW7 269.4 mm to (-231.5, 135.2)
- moved SW8 269.4 mm to (-223.1, 135.2)
- moved SW13 269.4 mm to (-214.7, 144.5)
- moved SW17 269.4 mm to (-214.7, 153.8)
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Connections:
- SW10 pad 2: C1 -> C4
- SW11 pad 2: C2 -> C3
- SW12 pad 2: C3 -> C2
- SW13 pad 2: C4 -> C1
- SW14 pad 2: C1 -> C4
- SW15 pad 2: C2 -> C3
- SW16 pad 2: C3 -> C2
- SW17 pad 2: C4 -> C1
- SW2 pad 2: C1 -> C4
- SW3 pad 2: C2 -> C3
- SW4 pad 2: C3 -> C2
- SW5 pad 2: C4 -> C1
- SW6 pad 2: C1 -> C4
- SW7 pad 2: C2 -> C3
- SW8 pad 2: C3 -> C2
- SW9 pad 2: C4 -> C1
Routing:
- net +5V: track 46.7 -> 328.0 mm, vias 0 -> 1
- net C4: track 33.7 -> 117.7 mm
- net L1: track 48.4 -> 130.6 mm
- net C3: track 33.7 -> 109.0 mm
- net L2: track 48.4 -> 122.0 mm
- net C2: track 33.7 -> 100.4 mm
- net L3: track 48.4 -> 113.3 mm
- net C1: track 33.7 -> 91.8 mm
- net L4: track 48.4 -> 104.7 mm
- net Net-(J12-Pin_1): track 0.00 -> 39.1 mm
- net Net-(J10-Pin_1): track 0.00 -> 34.6 mm, vias 0 -> 1
- net Net-(J13-Pin_1): track 0.00 -> 33.6 mm
- net ADC0: track 0.00 -> 28.9 mm
- net ADC1: track 0.00 -> 25.7 mm
- net A0: track 0.00 -> 24.1 mm
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
Commit message: Finaliza a organização dos componentes na PCB, ajusta footprints
Parts:
- C1, C2, C22, C23, C24, C4, C5: moved to B.Cu
- C18, C20, C21: footprint Capacitor_THT:CP_Radial_D4.0mm_P2.00mm -> Capacitor_SMD:C_0805_2012Metric; moved to B.Cu
- C19: footprint Capacitor_THT:CP_Radial_D4.0mm_P2.00mm -> Capacitor_SMD:C_0805_2012Metric
- C6, C7, C8, C9: footprint Capacitor_THT:CP_Radial_D4.0mm_P1.50mm -> Capacitor_SMD:C_0805_2012Metric; moved to B.Cu
- J9: footprint Connector_PinHeader_2.54mm:PinHeader_2x05_P2.54mm_Vertical -> Connector_IDC:IDC-Header_2x05_P2.54mm_Vertical
- R1, R22, R24, R25, R26: footprint Resistor_THT:R_Axial_DIN0207_L6.3mm_D2.5mm_P7.62mm_Horizontal -> Resistor_SMD:R_0805_2012Metric
- R23: footprint Resistor_THT:R_Axial_DIN0207_L6.3mm_D2.5mm_P7.62mm_Horizontal -> Resistor_SMD:R_0805_2012Metric; moved to B.Cu
- SW1: value SW_MEC_5G -> SW_Omron_B3FS
- moved C16 454.9 mm to (-200.2, 214.8)
- moved C17 454.9 mm to (-200.1, 219.9)
- moved PS1 454.9 mm to (-197.8, 213.2)
- moved RV5 388.4 mm to (-196.3, 95.0), turned to 90 degrees
- moved R23 313.9 mm to (-117.5, 98.8), turned to -90 degrees
- moved C24 312.9 mm to (-233.6, 229.8)
- moved C22 303.8 mm to (-222.4, 221.2)
- moved U9 300.0 mm to (-234.5, 239.7), turned to 90 degrees
- moved C18 295.2 mm to (-225.6, 241.9)
- moved C19 294.5 mm to (-231.9, 243.7)
- moved C23 292.2 mm to (-217.1, 213.6)
- moved C20 288.5 mm to (-232.0, 242.6), turned to -90 degrees
- moved J11 286.5 mm to (-221.7, 250.5)
- moved U8 284.0 mm to (-213.6, 221.3), turned to 90 degrees
- moved C13 284.0 mm to (-211.3, 114.4)
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Connections:
- J9 pad 1: MOSI -> MISO
- J9 pad 5: RST -> MOSI
- J9 pad 9: MISO -> RST
- R22 pad 2: Net-(R22-Pad2) -> Net-(U7-A)
- SW1 pad 2: GND -> RST
- U7 pad 1: Net-(R22-Pad2) -> unconnected-(U7-NC-Pad1)
- U7 pad 2: unconnected-(U7-A-Pad2) -> Net-(U7-A)
Routing:
- net +5V: track 328.0 -> 570.1 mm, vias 1 -> 12
- net E: track 0.00 -> 114.1 mm, vias 0 -> 2
- net D7: track 0.00 -> 111.2 mm
- net D6: track 0.00 -> 109.5 mm
- net D5: track 0.00 -> 107.8 mm
- net D4: track 0.00 -> 106.1 mm
- net TX: track 0.00 -> 92.5 mm, vias 0 -> 2
- net Net-(U10-VO): track 3.89 -> 90.0 mm
- net RX: track 0.00 -> 69.9 mm, vias 0 -> 2
- net +5VD: track 2.36 -> 45.1 mm, vias 0 -> 4
- net RST: track 0.00 -> 36.2 mm, vias 0 -> 2
- net SCK: track 0.00 -> 21.3 mm
- net MOSI: track 0.00 -> 18.5 mm
- net Net-(U7-VO): track 0.00 -> 16.6 mm
- net Net-(U8-C): track 0.00 -> 14.2 mm
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Other:
- outline, holes or cut-outs redrawn
- board text removed: "K"
