File: pasta do projeto/_autosave-av3.kicad_pcb (KiCad board)
At the start: 2 copper layers, 180 x 180 mm, 120 parts, among them J1 Conn_01x03, J10 Conn_01x03, J11 DE9_Pins_MountingHoles, J12 Conn_01x03, J13 Conn_01x03, J14 Conn_01x03, J15 Conn_02x04_Odd_Even, J16 Screw_Terminal_01x03, J2 Conn_01x03, J3 Conn_01x03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

Commit message: Finalização do orçamento e das malhas
Parts:
- moved C1 0.99 mm to (150.1, 146.4)
- moved C2 0.79 mm to (154.2, 146.4)
Routing:
- net GND: track 78.2 -> 38.5 mm, vias 1 -> 2
- net GNDD: track 3.70 -> 0.00 mm
- net +5V: track 574.2 -> 572.1 mm
